File: hardware/inkclip.kicad_pcb (KiCad board)
At the start: 2 copper layers, 103.1 x 63.6 mm, 40 parts, among them J1 AFC07-S24ECC-00, J2 U254-051T-4BH83-F1S, J3 SWD, Q1 Si1308BDL, SW0 TS-1187A, U1 XC6206P332MR-G, U2 STM32F411CEU6, Y1 12M

Commit message: hardware: remove draft Edge.Cuts
Other:
- board size 103.1 x 63.6 mm -> 33.4 x 38.9 mm
